Commit message: deleted unsed folders and integrated realsense into the ardrone frame

File: tum_simulator/cvg_sim_gazebo/urdf/quadrotor_sensors.urdf.xacro (robot description, xacro)
@@ -14,15 +14,20 @@
       <origin xyz="-0.15 0.0 0.0" rpy="0 ${90*M_PI/180} 0"/>
     </xacro:sonar_sensor>
-    <!-- Hokuyo UTM-30LX mounted upside down below the quadrotor body
-    <xacro:include filename="$(find cvg_sim_gazebo)/urdf/sensors/hokuyo_utm30lx.urdf.xacro" />
+    <!-- Hokuyo UTM-30LX mounted upside down below the quadrotor body -->
+    <!--<xacro:include filename="$(find cvg_sim_gazebo)/urdf/sensors/hokuyo_utm30lx.urdf.xacro" />
     <xacro:hokuyo_utm30lx name="laser0" parent="base_link" ros_topic="scan" update_rate="40" ray_count="1081" min_angle="135" max_angle="-135">
       <origin xyz="0.0 0.0 0.08" rpy="${M_PI} 0 0"/>
-    </xacro:hokuyo_utm30lx>-->
+    </xacro:hokuyo_utm30lx> -->
+    <!--- Realsense rs200 camera -->
+    <xacro:include filename="$(find realsense_gazebo_plugin)/urdf/realsense-RS200.macro.xacro"/>
+    <xacro:realsense-rs200 prefix="" parent="base_link">
+        <origin xyz="0.21 0 0.01" rpy="0 0 0" />
+    </xacro:realsense-rs200>
     <!-- The following two cameras should be united to one! -->
     <!-- Forward facing camera -->
-    <xacro:include filename="$(find cvg_sim_gazebo)/urdf/sensors/generic_camera.urdf.xacro" />
+<!--     <xacro:include filename="$(find cvg_sim_gazebo)/urdf/sensors/generic_camera.urdf.xacro" />
     <xacro:generic_camera name="front" sim_name="ardrone" parent="base_link" update_rate="60" res_x="640" res_y="360" image_format="R8G8B8" hfov="${81*M_PI/180}">
       <origin xyz="0.21 0.0 0.01" rpy="0 0 0"/>
-    </xacro:generic_camera>
+    </xacro:generic_camera> -->
     <!-- Downward facing camera -->
     <xacro:include filename="$(find cvg_sim_gazebo)/urdf/sensors/generic_camera.urdf.xacro" />
